Commit message: Adding depth modality

File: atom_test_rgb_camera_calibration/urdf/initial_estimate.urdf.xacro (robot description, xacro)
@@ -10,5 +10,5 @@
     </xacro:sensor_astra>
     <!-- ADD charuco REMOVED FROM HERE TO BE SEEN AS A DIFFERENT OBJECT IN THE SIMULATION -->
-    <!-- <xacro:include filename="$(find tripod_rgb_rgb_description)/models/charuco5X5.urdf.xacro" /> -->
+    <!-- <xacro:include filename="$(find atom_test_rgb_camera_description)/models/charuco5X5.urdf.xacro" /> -->
     <material name="grey">
         <color rgba="0.7 0.7 0.7 1.0" />
@@ -20,5 +20,5 @@
             <origin xyz="0 0 0" rpy="0 0 0" />
             <geometry>
-                <mesh filename="package://tripod_rgb_rgb_description/meshes/tripod/tripod.dae" scale="0.04 0.04 0.04" />
+                <mesh filename="package://atom_test_rgb_camera_description/meshes/tripod/tripod.dae" scale="0.04 0.04 0.04" />
             </geometry>
             <material name="grey" />
@@ -27,5 +27,5 @@
             <origin xyz="0 0 0" rpy="0 0 0" />
             <geometry>
-                <mesh filename="package://tripod_rgb_rgb_description/meshes/tripod/tripod.dae" scale="0.04 0.04 0.04" />
+                <mesh filename="package://atom_test_rgb_camera_description/meshes/tripod/tripod.dae" scale="0.04 0.04 0.04" />
             </geometry>
         </collision>

File: atom_test_rgb_camera_description/urdf/optimized.urdf.xacro (robot description, xacro)
@@ -26,5 +26,5 @@
   </link>
   <joint name="camera_rgb_joint" type="fixed">
-    <origin xyz="0.0 -0.045 0.0" rpy="0.0 -0.0 0.0"/>
+    <origin xyz="0.00010158958797154281 -0.042953467785865576 -0.0015448842947527724" rpy="0.00046995312155169927 2.388714950993065e-05 0.0001895113226526851"/>
     <parent link="camera_link"/>
     <child link="camera_rgb_frame"/>
@@ -38,5 +38,5 @@
   <link name="camera_rgb_optical_frame"/>
   <joint name="camera_depth_joint" type="fixed">
-    <origin xyz="0.0 -0.02 0.0" rpy="0.0 0.0 0.0"/>
+    <origin xyz="-0.003349810132048032 -0.017969203137631305 0.0010404538331909893" rpy="-0.0014918535772643327 -0.00039341491478172744 8.162331229562133e-05"/>
     <parent link="camera_link"/>
     <child link="camera_depth_frame"/>
@@ -129,5 +129,5 @@
       <origin xyz="0.0 0.0 0.0" rpy="0.0 0.0 0.0"/>
       <geometry>
-        <mesh filename="package://tripod_rgb_rgb_description/meshes/tripod/tripod.dae" scale="0.04 0.04 0.04"/>
+        <mesh filename="package://atom_test_rgb_camera_description/meshes/tripod/tripod.dae" scale="0.04 0.04 0.04"/>
       </geometry>
       <material name="grey"/>
@@ -136,5 +136,5 @@
       <origin xyz="0.0 0.0 0.0" rpy="0.0 0.0 0.0"/>
       <geometry>
-        <mesh filename="package://tripod_rgb_rgb_description/meshes/tripod/tripod.dae" scale="0.04 0.04 0.04"/>
+        <mesh filename="package://atom_test_rgb_camera_description/meshes/tripod/tripod.dae" scale="0.04 0.04 0.04"/>
       </geometry>
     </collision>
